File: KiCAD Files/TVZSolderingPracticeKit.kicad_sch (KiCad schematic)
At the start: 0 parts

Commit message: update
Parts:
- added BT1: 9V, symbol Device:Battery_Cell
- added BZ1: Buzzer, symbol Device:Buzzer
- added C1: 100n, symbol Device:C
- added C2: C, symbol Device:C
- added D1: LED, symbol Device:LED
- added D2: D, symbol Device:D
- added H1, H2, H3, H4: MountingHole, symbol Mechanical:MountingHole
- added R1: 6k2, symbol Device:R
- added R10, R11, R12, R13, R14, R15, R16, R17, R18, R19: R, symbol Device:R
- added R2: 390, symbol Device:R
- added R3: 910, symbol Device:R
- added R4, R9: 1k, symbol Device:R
- added R5: 1k1, symbol Device:R
- added R6: 620, symbol Device:R
- added R7: 1k3, symbol Device:R
- added R8: 1k5, symbol Device:R
- added RV1: R_Potentiometer, symbol Device:R_Potentiometer
- added SW1, SW2, SW3, SW4, SW5, SW6, SW7, SW8: SW_Push, symbol Switch:SW_Push
- added SW9: SW_SPST, symbol Switch:SW_SPST
- added U1: NE555P, Package_DIP:DIP-8_W7.62mm, symbol Timer:NE555P
Connections:
- new net: R1.1, R9.1, U1.7 (DIS)
- new net: R9.2, SW9.2 (B), U1.4 (R), U1.8 (VCC)
- new net: R10.1, R11.1, R12.1, R13.1, R14.1, R15.1, R16.1, R17.1, R18.1, R19.1
- new net: R7.2, R8.1, SW7.2
- new net: R8.2, SW8.2
- new net: C1.1, SW1.1, SW2.1, SW3.1, SW4.1, SW5.1, SW6.1, SW7.1, SW8.1, U1.2 (TR), U1.6 (THR)
- new net: R3.2, R4.1, SW3.2
- new net: R1.2, R2.1, SW1.2
- new net: R2.2, R3.1, SW2.2
- new net: BZ1.1 (+), U1.3 (Q)
- new net: R5.2, R6.1, SW5.2
- new net: R6.2, R7.1, SW6.2
- new net: BT1.1 (+), SW9.1 (A)
- new net: R4.2, R5.1, SW4.2
- new net GND1: BT1.2 (-), BZ1.2 (-), C1.2, U1.1 (GND)
- new net GND2: R10.2, R11.2, R12.2, R13.2, R14.2, R15.2, R16.2, R17.2, R18.2, R19.2
- no-connect marks 0 -> 1
Other:
- note added: "PIANO"

Commit message: update
Parts:
- added R20, R21, R22, R23, R24, R25: R, Resistor_THT:R_Axial_DIN0207_L6.3mm_D2.5mm_P7.62mm_Horizontal, symbol Device:R
- H1, H2, H3, H4: footprint (none) -> MountingHole:MountingHole_3.2mm_M3
- R10, R11, R12, R13, R14: footprint (none) -> Resistor_THT:R_Axial_DIN0207_L6.3mm_D2.5mm_P2.54mm_Vertical
- R15, R16, R17, R18, R19: footprint (none) -> Resistor_THT:R_Axial_DIN0207_L6.3mm_D2.5mm_P7.62mm_Horizontal
Connections:
- new net: R20.1, R21.1, R22.1, R23.1, R24.1, R25.1
- new net GND3: R20.2, R21.2, R22.2, R23.2, R24.2, R25.2
Other:
- moved on the sheet: D1, RV1

Commit message: update
Parts:
- removed C2: C, symbol Device:C
- removed D1: LED, symbol Device:LED
- removed D2: D, symbol Device:D
- removed H1, H2, H3, H4: MountingHole, MountingHole:MountingHole_3.2mm_M3, symbol Mechanical:MountingHole
- removed R10, R11, R12, R13, R14: R, Resistor_THT:R_Axial_DIN0207_L6.3mm_D2.5mm_P2.54mm_Vertical, symbol Device:R
- removed R15, R16, R17, R18, R19, R20, R21, R22, R23, R24, R25: R, Resistor_THT:R_Axial_DIN0207_L6.3mm_D2.5mm_P7.62mm_Horizontal, symbol Device:R
- removed RV1: R_Potentiometer, symbol Device:R_Potentiometer

Commit message: update
Parts:
- removed SW9: SW_SPST, symbol Switch:SW_SPST
- added SW10: SW_SPDT, Footprint:OS102011MS2QN1, symbol Switch:SW_SPDT
- BZ1: footprint (none) -> Footprint:LD-BZEN-1205
- R1, R2, R3, R4, R5, R6, R7, R8, R9: footprint (none) -> Resistor_THT:R_Axial_DIN0207_L6.3mm_D2.5mm_P7.62mm_Horizontal
Connections:
- net at R9.2, U1.4 (R), U1.8 (VCC): now also SW10.1 (A)
- net at BT1.1 (+): now also SW10.2 (B)
- no-connect marks 1 -> 2

Commit message: update
Parts:
- R1, R2, R3, R4, R5, R6, R7, R8, R9: footprint Resistor_THT:R_Axial_DIN0207_L6.3mm_D2.5mm_P7.62mm_Horizontal -> Resistor_THT:R_Axial_DIN0207_L6.3mm_D2.5mm_P10.16mm_Horizontal
Connections:
- net at R7.2, R8.1: now also SW2.1; no longer SW7.2
- net at R8.2: now also SW1.1; no longer SW8.2
- net at R3.2, R4.1: now also SW6.1; no longer SW3.2
- net at R1.2, R2.1: now also SW8.1; no longer SW1.2
- net at R2.2, R3.1: now also SW7.1; no longer SW2.2
- net at R5.2, R6.1: now also SW4.1; no longer SW5.2
- net at R6.2, R7.1: now also SW3.1; no longer SW6.2
- net at R4.2, R5.1: now also SW5.1; no longer SW4.2
- new net: C1.1, SW1.2, SW2.2, SW3.2, SW4.2, SW5.2, SW6.2, SW7.2, SW8.2, U1.2 (TR), U1.6 (THR)
Other:
- note added: "Najniža nota"
- note added: "Najviša nota"
- moved on the sheet: BT1, BZ1, C1, R1, R2, R3, R4, R5, R6, R7, R8, R9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

Commit message: update
Parts:
- removed BT1: 9V, symbol Device:Battery_Cell
- added D1: SR150-DC, Diode_THT:D_DO-41_SOD81_P10.16mm_Horizontal, symbol Device:D_Schottky
- added J1: Barrel Jack, Footprint:DCJ250-10-A-K1-K, symbol Connector:Barrel_Jack_MountingPin
- added U2: ~, symbol Symbols:ICVT-8P
- BZ1: value Buzzer -> LD-BZEN-1205; TME Part Number (none) -> LD-BZEN-1205
- C1: footprint (none) -> Capacitor_THT:C_Disc_D3.0mm_W1.6mm_P2.50mm; TME Part Number (none) -> CCT-100N/50V-S
- R1: TME Part Number (none) -> 1/4W6.2K
- R2: TME Part Number (none) -> CF1/4W-390R
- R3: TME Part Number (none) -> 1/4W910R
- R4, R9: TME Part Number (none) -> 1/4W1.0K
- R5: TME Part Number (none) -> 1/4W1.1K
- R6: TME Part Number (none) -> 1/4W620R
- R7: TME Part Number (none) -> 1/4W1.3K
- R8: TME Part Number (none) -> 1/4W1.5K
- SW1, SW2, SW3, SW4, SW5, SW6, SW7, SW8: footprint (none) -> Button_Switch_THT:SW_PUSH_6mm_H4.3mm; TME Part Number (none) -> TACT-64K-F
- U1: footprint Package_DIP:DIP-8_W7.62mm -> Footprint:DIP-8_W7.62mm-socket; TME Part Number (none) -> NE555P
Connections:
- net GND1: now also J1.2
- net at R9.2, U1.4 (R), U1.8 (VCC): now also D1.1 (K); no longer SW10.1 (A)
- net at SW10.2 (B): now also J1.1
- new net: D1.2 (A), SW10.1 (A)
- no-connect marks 2 -> 3
Other:
- note added: "TO-DO: - obojati switch - buzzer model fix"
- moved on the sheet: SW10

Commit message: update
Parts:
- added H1, H2, H3, H4: MountingHole_Pad, MountingHole:MountingHole_3.2mm_M3_Pad_Via, symbol Mechanical:MountingHole_Pad
Connections:
- no-connect marks 3 -> 7
Other:
- note removed: "TO-DO: - obojati switch - buzzer model fix"

Commit message: update
Parts:
- added C2: 470u / 50V, Capacitor_THT:CP_Radial_D10.0mm_P5.00mm, symbol Device:C_Polarized
- added D2: RED, LED_THT:LED_D5.0mm, symbol Device:LED
- added D3: YELLOW, LED_THT:LED_D5.0mm, symbol Device:LED
- added D4: GREEN, LED_THT:LED_D5.0mm, symbol Device:LED
- added J2: Conn_01x05_Pin, Connector_PinHeader_2.54mm:PinHeader_1x05_P2.54mm_Horizontal, symbol Connector:Conn_01x05_Pin
- added J3: Conn_01x05_Socket, Connector_PinSocket_2.54mm:PinSocket_1x05_P2.54mm_Vertical, symbol Connector:Conn_01x05_Socket
- added J4, J5: Conn_01x03_Pin, Connector_PinHeader_2.54mm:PinHeader_1x03_P2.54mm_Vertical, symbol Connector:Conn_01x03_Pin
- added R10: 4k7, Resistor_THT:R_Axial_DIN0207_L6.3mm_D2.5mm_P10.16mm_Horizontal, symbol Device:R
- added R11: 2k2, Resistor_THT:R_Axial_DIN0207_L6.3mm_D2.5mm_P10.16mm_Horizontal, symbol Device:R
- added R12, R13, R14: 2k2, Resistor_THT:R_Axial_DIN0207_L6.3mm_D2.5mm_P2.54mm_Vertical, symbol Device:R
- added SW11: C/D, Footprint:OS102011MS2QN1, symbol Switch:SW_SPDT
- added TP1, TP2: TestPoint, Footprint:Wire, symbol Connector:TestPoint
- SW10: value SW_SPDT -> POWER
- renumbered R8 to R1, R7 to R2, R6 to R3, R5 to R4, R4 to R5, R3 to R6, R2 to R7, R1 to R8
Connections:
- net GND1: now also D3.1 (K), D4.2 (A), J2.2 (Pin_2), J2.4 (Pin_4), J3.2 (Pin_2), J3.4 (Pin_4), J4.1 (Pin_1), J4.3 (Pin_3), J5.1 (Pin_1), J5.3 (Pin_3), R10.1, R12.1, R13.1, R14.1, SW11.3 (C)
- net VDD: now reaches D1.1 (K), R9.2, U1.4 (R), U1.8 (VCC)
- net VDD: now also D2.2 (A), SW11.1 (A)
- new net: R12.2, R13.2, R14.2
- new net: C2.2, D3.2 (A), D4.1 (K)
- new net: D2.1 (K), R10.2
- new net: C2.1, R11.1
- new net: R11.2, SW11.2 (B)
- no-connect marks 7 -> 17
Other:
- note added: "CHARGE"
- note added: "DISCHARGE"
- note added: "TODO: - dummy potenciometar - dodati tme komponente u BOM - Jumperi u BOM odnosno dodati na shemi"
- moved on the sheet: D1, J1, SW10
