File: KiCAD Files/TVZSolderingPracticeKit.kicad_sch (KiCad schematic)
At the start: 44 parts, among them J1 Barrel Jack, J2 Conn_01x05_Pin, J3 Conn_01x05_Socket, J4 Conn_01x03_Pin, J5 Conn_01x03_Pin, SW1 SW_Push, SW10 POWER, SW11 C/D, SW2 SW_Push, SW3 SW_Push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

Commit message: Update TVZSolderingPracticeKit.kicad_sch
Other:
- note added: "TODO: - dummy potenciometar RK09K1130AH1 - dodati tme komponente u BOM - Jumperi u BOM odnosno dodati na shemi"
- note removed: "TODO: - dummy potenciometar - dodati tme komponente u BOM - Jumperi u BOM odnosno dodati na shemi"
Changed lines of the file:
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@@
 	(generator_version "9.0")
 	(paper "A4")
-	(text "TODO:\n- dummy potenciometar\n- dodati tme komponente u BOM\n- Jumperi u BOM odnosno dodati na shemi\n"
+	(text "TODO:\n- dummy potenciometar RK09K1130AH1\n- dodati tme komponente u BOM\n- Jumperi u BOM odnosno dodati na shemi\n"
 		(exclude_from_sim no)
 		(at 86.614 174.498 0)

Commit message: update
Other:
- note added: "TODO: - ispraviti dimenzije pločice - dummy potenciometar RK09K1130AH1 - dodati tme komponente u BOM - Jumperi u BOM odnosno dodati na shemi"
- note removed: "TODO: - dummy potenciometar RK09K1130AH1 - dodati tme komponente u BOM - Jumperi u BOM odnosno dodati na shemi"
Changed lines of the file:
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@@
 	(generator_version "9.0")
 	(paper "A4")
-	(text "TODO:\n- dummy potenciometar RK09K1130AH1\n- dodati tme komponente u BOM\n- Jumperi u BOM odnosno dodati na shemi\n"
+	(text "TODO:\n- ispraviti dimenzije pločice\n- dummy potenciometar RK09K1130AH1\n- dodati tme komponente u BOM\n- Jumperi u BOM odnosno dodati na shemi\n"
 		(exclude_from_sim no)
 		(at 86.614 174.498 0)

Commit message: Update TVZSolderingPracticeKit.kicad_sch
Other:
- note added: "TODO: - ispraviti dimenzije pločice i napraviti zube s dvije strane - dummy potenciometar RK09K1130AH1 - dodati tme komponente u BOM - Jumperi u BOM odnosno dodati na shemi"
- note removed: "TODO: - ispraviti dimenzije pločice - dummy potenciometar RK09K1130AH1 - dodati tme komponente u BOM - Jumperi u BOM odnosno dodati na shemi"
Changed lines of the file:
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@@
 	(generator_version "9.0")
 	(paper "A4")
-	(text "TODO:\n- ispraviti dimenzije pločice\n- dummy potenciometar RK09K1130AH1\n- dodati tme komponente u BOM\n- Jumperi u BOM odnosno dodati na shemi\n"
+	(text "TODO:\n- ispraviti dimenzije pločice i napraviti zube s dvije strane\n- dummy potenciometar RK09K1130AH1\n- dodati tme komponente u BOM\n- Jumperi u BOM odnosno dodati na shemi\n"
 		(exclude_from_sim no)
 		(at 86.614 174.498 0)

Commit message: update
Other:
- note added: "TODO: - ispraviti dimenzije pločice i napraviti zube s dvije strane - dummy potenciometar RK09K1130AH1 - dodati tme komponente u BOM - Jumperi u BOM odnosno dodati na shemi - 3d printatni dio s držačem za bateriju"
- note removed: "TODO: - ispraviti dimenzije pločice i napraviti zube s dvije strane - dummy potenciometar RK09K1130AH1 - dodati tme komponente u BOM - Jumperi u BOM odnosno dodati na shemi"
Changed lines of the file:
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@@
 	(generator_version "9.0")
 	(paper "A4")
-	(text "TODO:\n- ispraviti dimenzije pločice i napraviti zube s dvije strane\n- dummy potenciometar RK09K1130AH1\n- dodati tme komponente u BOM\n- Jumperi u BOM odnosno dodati na shemi\n"
+	(text "TODO:\n- ispraviti dimenzije pločice i napraviti zube s dvije strane\n- dummy potenciometar RK09K1130AH1\n- dodati tme komponente u BOM\n- Jumperi u BOM odnosno dodati na shemi\n- 3d printatni dio s držačem za bateriju\n"
 		(exclude_from_sim no)
 		(at 86.614 174.498 0)

Commit message: update
Other:
- note added: "TODO: - dummy potenciometar RK09K1130AH1 - dodati tme komponente u BOM - Jumperi u BOM odnosno dodati na shemi - 3d printatni dio s držačem za bateriju - JLCJLCJLCJLC"
- note removed: "TODO: - ispraviti dimenzije pločice i napraviti zube s dvije strane - dummy potenciometar RK09K1130AH1 - dodati tme komponente u BOM - Jumperi u BOM odnosno dodati na shemi - 3d printatni dio s držačem za bateriju"
Changed lines of the file:
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@@
 	(generator_version "9.0")
 	(paper "A4")
-	(text "TODO:\n- ispraviti dimenzije pločice i napraviti zube s dvije strane\n- dummy potenciometar RK09K1130AH1\n- dodati tme komponente u BOM\n- Jumperi u BOM odnosno dodati na shemi\n- 3d printatni dio s držačem za bateriju\n"
+	(text "TODO:\n- dummy potenciometar RK09K1130AH1\n- dodati tme komponente u BOM\n- Jumperi u BOM odnosno dodati na shemi\n- 3d printatni dio s držačem za bateriju\n- JLCJLCJLCJLC\n"
 		(exclude_from_sim no)
 		(at 86.614 174.498 0)

Commit message: update
Parts:
- added D5: WHITE, LED_THT:LED_D5.0mm, symbol Device:LED
- added R15: 2k2, Resistor_THT:R_Axial_DIN0207_L6.3mm_D2.5mm_P10.16mm_Horizontal, symbol Device:R
- added RV1: 10k, Footprint:RK09K1130AH1, symbol Device:R_Potentiometer
Connections:
- net GND1: now also D5.1 (K)
- net VDD: now also RV1.3
- new net: D5.2 (A), R15.1
- new net: R15.2, RV1.2
- no-connect marks 17 -> 18
Other:
- note added: "TODO: - dummy potenciometar RK09K1130AH1 - dodati tme komponente u BOM - Jumperi u BOM odnosno dodati na shemi - 3d printatni dio s držačem za bateriju - jumperi 3d modeli - JLCJLCJLCJLC"
- note removed: "TODO: - dummy potenciometar RK09K1130AH1 - dodati tme komponente u BOM - Jumperi u BOM odnosno dodati na shemi - 3d printatni dio s držačem za bateriju - JLCJLCJLCJLC"

Commit message: update
Parts:
- added J6: JUMPER-H/R, symbol Symbols:Jumper
- added J7: JUMPER-H/B, symbol Symbols:Jumper
- J2: TME Part Number (none) -> PH1RB-40-UA
- J3: TME Part Number (none) -> ZL262-5SG
- J4, J5: TME Part Number (none) -> ZL201-03G
- TP1, TP2: now left out of the parts list
Other:
- note added: "TODO: - Jumperi u BOM odnosno dodati na shemi - 3d printatni dio s držačem za bateriju - jumperi 3d modeli"
- note removed: "TODO: - dummy potenciometar RK09K1130AH1 - dodati tme komponente u BOM - Jumperi u BOM odnosno dodati na shemi - 3d printatni dio s držačem za bateriju - jumperi 3d modeli - JLCJLCJLCJLC"
Changed lines of the file:
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@@
 	(generator_version "9.0")
 	(paper "A4")
-	(text "TODO:\n- dummy potenciometar RK09K1130AH1\n- dodati tme komponente u BOM\n- Jumperi u BOM odnosno dodati na shemi\n- 3d printatni dio s držačem za bateriju\n- jumperi 3d modeli\n- JLCJLCJLCJLC\n"
+	(text "TODO:\n- Jumperi u BOM odnosno dodati na shemi\n- 3d printatni dio s držačem za bateriju\n- jumperi 3d modeli\n"
 		(exclude_from_sim no)
 		(at 86.614 174.498 0)
@@
 			)
 		)
+		(property "TME Part Number" "PH1RB-40-UA"
+			(at 43.18 87.63 0)
+			(effects
+				(font
+					(size 1.27 1.27)
+				)
+				(hide yes)
+			)
+		)
 		(pin "3"
 		)
@@
 			)
 		)
+		(property "TME Part Number" "ZL201-03G"
+			(at 43.18 132.08 0)
+			(effects
+				(font
+					(size 1.27 1.27)
+				)
+				(hide yes)
+			)
+		)
 		(pin "2"
 		)
@@
 		(unit 1)
 		(exclude_from_sim no)
-		(in_bom yes)
+		(in_bom no)
 		(on_board yes)
 		(dnp no)
@@
 	)
 	(symbol
+		(lib_id "Symbols:Jumper")
+		(at 21.59 111.76 0)
+		(unit 1)
+		(exclude_from_sim no)
+		(in_bom yes)
+		(on_board no)
+		(dnp no)
+		(fields_autoplaced yes)
+		(property "Reference" "J6"
+			(at 26.67 107.9499 0)
+			(effects
+				(font
+					(size 1.27 1.27)
+				)
+				(justify left)
+			)
+		)
+		(property "Value" "JUMPER-H/R"
+			(at 26.67 110.4899 0)
+			(effects
+				(font
+					(size 1.27 1.27)
+				)
+				(justify left)
+			)
+		)
+		(property "Footprint" ""
+			(at 21.59 111.76 0)
+			(effects
+				(font
+					(size 1.27 1.27)
+				)
+				(hide yes)
+			)
+		)
+		(property "Datasheet" ""
+			(at 21.59 111.76 0)
+			(effects
+				(font
+					(size 1.27 1.27)
+				)
+				(hide yes)
+			)
+		)
+		(property "Description" ""
+			(at 21.59 111.76 0)
+			(effects
+				(font
+					(size 1.27 1.27)
+				)
+				(hide yes)
+			)
+		)
+		(property "TME Part Number" "JUMPER-H/R"
+			(at 21.59 111.76 0)
+			(effects
+				(font
+					(size 1.27 1.27)
+				)
+				(hide yes)
+			)
+		)
+		(instances
+			(project ""
+				(path "/f8b435ab-5f6e-4fa9-ab74-0f98728395bc"
+					(reference "J6")
+					(unit 1)
+				)
+			)
+		)
+	)
+	(symbol
 		(lib_id "power:GND1")
 		(at 151.13 53.34 0)
@@
 	)
 	(symbol
+		(lib_id "Symbols:Jumper")
+		(at 21.59 134.62 0)
+		(unit 1)
+		(exclude_from_sim no)
+		(in_bom yes)
+		(on_board no)
+		(dnp no)
+		(fields_autoplaced yes)
+		(property "Reference" "J7"
+			(at 26.67 130.8099 0)
+			(effects
+				(font
+					(size 1.27 1.27)
+				)
+				(justify left)
+			)
+		)
+		(property "Value" "JUMPER-H/B"
+			(at 26.67 133.3499 0)
+			(effects
+				(font
+					(size 1.27 1.27)
+				)
+				(justify left)
+			)
+		)
+		(property "Footprint" ""
+			(at 21.59 134.62 0)
+			(effects
+				(font
+					(size 1.27 1.27)
+				)
+				(hide yes)
+			)
+		)
+		(property "Datasheet" ""
+			(at 21.59 134.62 0)
+			(effects
+				(font
+					(size 1.27 1.27)
+				)
+				(hide yes)
+			)
+		)
+		(property "Description" ""
+			(at 21.59 134.62 0)
+			(effects
+				(font
+					(size 1.27 1.27)
+				)
+				(hide yes)
+			)
+		)
+		(property "TME Part Number" "JUMPER-H/B"
+			(at 21.59 134.62 0)
+			(effects
+				(font
+					(size 1.27 1.27)
+				)
+				(hide yes)
+			)
+		)
+		(instances
+			(project "TVZSolderingPracticeKit"
+				(path "/f8b435ab-5f6e-4fa9-ab74-0f98728395bc"
+					(reference "J7")
+					(unit 1)
+				)
+			)
+		)
+	)
+	(symbol
 		(lib_id "Connector:Conn_01x03_Pin")
 		(at 43.18 110.49 0)
@@
 			)
 		)
+		(property "TME Part Number" "ZL201-03G"
+			(at 43.18 110.49 0)
+			(effects
+				(font
+					(size 1.27 1.27)
+				)
+				(hide yes)
+			)
+		)
 		(pin "2"
 		)
@@
 		(unit 1)
 		(exclude_from_sim no)
-		(in_bom yes)
+		(in_bom no)
 		(on_board yes)
 		(dnp no)
@@
 			(at 69.85 87.63 0)
 			(effects
+				(font
+					(size 1.27 1.27)
+				)
+				(hide yes)
+			)
+		)
+		(property "TME Part Number" "ZL262-5SG"
+			(at 69.85 87.63 0)
+			(effects

Commit message: update
Connections:
- net at RV1.1: now also R15.2, RV1.2
- no-connect marks 18 -> 17
Other:
- note added: "TODO: - promijeniti 3d modele LEDica da budu realne boje - 3d printatni dio s držačem za bateriju - urediti shemu, montažnu shemu i BOM - urediti github - napisati upute za sastavljanje - dodati u bom mehaničke komponente za 3D printani dio (vijke i matice)"
- note removed: "TODO: - Jumperi u BOM odnosno dodati na shemi - 3d printatni dio s držačem za bateriju - jumperi 3d modeli"
Changed lines of the file:
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@@
 	(generator_version "9.0")
 	(paper "A4")
-	(text "TODO:\n- Jumperi u BOM odnosno dodati na shemi\n- 3d printatni dio s držačem za bateriju\n- jumperi 3d modeli\n"
+	(text "TODO:\n- promijeniti 3d modele LEDica da budu realne boje\n- 3d printatni dio s držačem za bateriju\n- urediti shemu, montažnu shemu i BOM\n- urediti github\n- napisati upute za sastavljanje\n- dodati u bom mehaničke komponente za 3D printani dio (vijke i matice)"
 		(exclude_from_sim no)
 		(at 86.614 174.498 0)
@@
 	)
 	(junction
+		(at 148.59 125.73)
+		(diameter 0)
+		(color 0 0 0 0)
+	)
+	(junction
 		(at 118.11 62.23)
 		(diameter 0)
@@
 	)
 	(no_connect
-		(at 146.05 125.73)
-	)
-	(no_connect
 		(at 64.77 87.63)
 	)
@@
 		)
 		(stroke
+			(width 0)
+			(type default)
+		)
+	)
+	(wire
+		(pts
+			(xy 146.05 125.73) (xy 148.59 125.73)
+		)
+		(stroke
