File: KiCAD Files/TVZSolderingPracticeKit.kicad_sch (KiCad schematic)
At the start: 49 parts, among them J1 Barrel Jack, J2 Conn_01x05_Pin, J3 Conn_01x05_Socket, J4 Conn_01x03_Pin, J5 Conn_01x03_Pin, J6 JUMPER-H/R, J7 JUMPER-H/B, SW1 SW_Push, SW10 POWER, SW11 C/D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

Commit message: update
Other:
- note added: "TODO: - promijeniti 3d modele LEDica da budu realne boje - 3d printatni dio s držačem za bateriju - urediti shemu, montažnu shemu i BOM - dodati baterije u BOM - urediti github - napisati upute za sastavljanje - dodati u bom mehaničke komponente za 3D printani dio (vijke i matice)"
- note removed: "TODO: - promijeniti 3d modele LEDica da budu realne boje - 3d printatni dio s držačem za bateriju - urediti shemu, montažnu shemu i BOM - urediti github - napisati upute za sastavljanje - dodati u bom mehaničke komponente za 3D printani dio (vijke i matice)"
Changed lines of the file:
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@@
 	(generator_version "9.0")
 	(paper "A4")
-	(text "TODO:\n- promijeniti 3d modele LEDica da budu realne boje\n- 3d printatni dio s držačem za bateriju\n- urediti shemu, montažnu shemu i BOM\n- urediti github\n- napisati upute za sastavljanje\n- dodati u bom mehaničke komponente za 3D printani dio (vijke i matice)"
+	(text "TODO:\n- promijeniti 3d modele LEDica da budu realne boje\n- 3d printatni dio s držačem za bateriju\n- urediti shemu, montažnu shemu i BOM\n- dodati baterije u BOM\n- urediti github\n- napisati upute za sastavljanje\n- dodati u bom mehaničke komponente za 3D printani dio (vijke i matice)"
 		(exclude_from_sim no)
 		(at 86.614 174.498 0)

Commit message: update
Parts:
- added U3: ~, symbol Symbols:BAT
Other:
- note added: "9V BATTERY"
- note added: "CAPACITOR CHARGE/DISCHARGE"
- note added: "DIP8 socket"
- note added: "DUMMY COMPONENTS"
- note added: "High frequency note"
- note added: "Low frequency note"
- note added: "MALE AND FEMALE HEADERS"
- note added: "MALE HEADERS WITH JUMPERS"
- note added: "MECHANICAL"
- note added: "NOTES: - dodati u bom mehaničke komponente za 3D printani dio (vijke i matice) - urediti github - napisati upute za sastavljanje (koristeći ibom)"
- note added: "POTENTIOMETER WITH LED"
- note added: "RESISTORS"
- note removed: "Najniža nota"
- note removed: "Najviša nota"
- note removed: "TODO: - promijeniti 3d modele LEDica da budu realne boje - 3d printatni dio s držačem za bateriju - urediti shemu, montažnu shemu i BOM - dodati baterije u BOM - urediti github - napisati upute za sastavljanje - dodati u bom mehaničke komponente za 3D printani dio (vijke i matice)"
- moved on the sheet: BZ1, C1, C2, D1, D2, D3, D4, D5, H1, H2, H3, H4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

Commit message: update
Parts:
- added U10, U11, U8, U9: ~, symbol Symbols:B3/BN116
- added U4, U5, U6, U7: ~, symbol Symbols:B2.5X5/BN2724
Other:
- note added: "B2.5X5/BN2724 screws"
- note added: "B3/BN116 nuts"
- note removed: "NOTES: - dodati u bom mehaničke komponente za 3D printani dio (vijke i matice) - urediti github - napisati upute za sastavljanje (koristeći ibom)"
- moved on the sheet: H1, H2, H3, H4, TP1, TP2

Commit message: update
Parts:
- C1: TME Part Number CCT-100N/50V-S -> C320C104K5R5TA7317
Changed lines of the file:
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@@
 			)
 		)
-		(property "TME Part Number" "CCT-100N/50V-S"
+		(property "TME Part Number" "C320C104K5R5TA7317"
 			(at 168.91 69.85 0)
 			(effects
