File: KiCAD Files/TVZSolderingPracticeKit.kicad_pcb (KiCad board)
At the start: 2 copper layers, 100 x 100 mm, 0 parts

Commit message: update
Parts:
- added H1: MountingHole, MountingHole:MountingHole_3.2mm_M3, F.Cu at (90.0, 49.5)
- added H2: MountingHole, MountingHole:MountingHole_3.2mm_M3, F.Cu at (183.0, 49.5)
- added H3: MountingHole, MountingHole:MountingHole_3.2mm_M3, F.Cu at (183.0, 142.5)
- added H4: MountingHole, MountingHole:MountingHole_3.2mm_M3, F.Cu at (90.0, 142.5)
- added R10: R, Resistor_THT:R_Axial_DIN0207_L6.3mm_D2.5mm_P2.54mm_Vertical, F.Cu at (101.0, 55.0)
- added R11: R, Resistor_THT:R_Axial_DIN0207_L6.3mm_D2.5mm_P2.54mm_Vertical, F.Cu at (101.0, 60.0)
- added R12: R, Resistor_THT:R_Axial_DIN0207_L6.3mm_D2.5mm_P2.54mm_Vertical, F.Cu at (101.0, 65.0)
- added R13: R, Resistor_THT:R_Axial_DIN0207_L6.3mm_D2.5mm_P2.54mm_Vertical, F.Cu at (101.0, 70.0)
- added R14: R, Resistor_THT:R_Axial_DIN0207_L6.3mm_D2.5mm_P2.54mm_Vertical, F.Cu at (101.0, 75.0)
- added R15: R, Resistor_THT:R_Axial_DIN0207_L6.3mm_D2.5mm_P7.62mm_Horizontal, F.Cu at (107.9, 55.0)
- added R16: R, Resistor_THT:R_Axial_DIN0207_L6.3mm_D2.5mm_P7.62mm_Horizontal, F.Cu at (107.9, 60.0)
- added R17: R, Resistor_THT:R_Axial_DIN0207_L6.3mm_D2.5mm_P7.62mm_Horizontal, F.Cu at (107.9, 65.0)
- added R18: R, Resistor_THT:R_Axial_DIN0207_L6.3mm_D2.5mm_P7.62mm_Horizontal, F.Cu at (107.9, 70.0)
- added R19: R, Resistor_THT:R_Axial_DIN0207_L6.3mm_D2.5mm_P7.62mm_Horizontal, F.Cu at (107.9, 75.0)
- added R20: R, Resistor_THT:R_Axial_DIN0207_L6.3mm_D2.5mm_P7.62mm_Horizontal, F.Cu at (122.5, 62.6)
- added R21: R, Resistor_THT:R_Axial_DIN0207_L6.3mm_D2.5mm_P7.62mm_Horizontal, F.Cu at (122.5, 67.4)
- added R22: R, Resistor_THT:R_Axial_DIN0207_L6.3mm_D2.5mm_P7.62mm_Horizontal, F.Cu at (127.5, 62.6)
- added R23: R, Resistor_THT:R_Axial_DIN0207_L6.3mm_D2.5mm_P7.62mm_Horizontal, F.Cu at (127.5, 67.4)
- added R24: R, Resistor_THT:R_Axial_DIN0207_L6.3mm_D2.5mm_P7.62mm_Horizontal, F.Cu at (132.5, 62.6)
- added R25: R, Resistor_THT:R_Axial_DIN0207_L6.3mm_D2.5mm_P7.62mm_Horizontal, F.Cu at (132.5, 67.4)
- added U1: NE555P, Package_DIP:DIP-8_W7.62mm, F.Cu at (135.4, 97.9)
Routing:
- net Net-(R10-Pad1): track 0.00 -> 46.8 mm
- net Net-(R20-Pad1): track 0.00 -> 24.8 mm
- added copper zone on B.Cu, net GND2
- added copper zone on F.Cu, net GND2
- added copper zone on B.Cu, net GND3
- added copper zone on F.Cu, net GND3
Other:
- outline, holes or cut-outs redrawn
- board text added: "Solid pad"
- board text added: "Thermal reliefs"

Commit message: update
Parts:
- removed H1, H2, H3, H4: MountingHole, MountingHole:MountingHole_3.2mm_M3
- removed R10, R11, R12, R13, R14: R, Resistor_THT:R_Axial_DIN0207_L6.3mm_D2.5mm_P2.54mm_Vertical
- removed R15, R16, R17, R18, R19, R20, R21, R22, R23, R24, R25: R, Resistor_THT:R_Axial_DIN0207_L6.3mm_D2.5mm_P7.62mm_Horizontal
- moved U1 19.0 mm to (151.9, 88.4)
Routing:
- net Net-(R10-Pad1): track 46.8 -> 0.00 mm
- net Net-(R20-Pad1): track 24.8 -> 0.00 mm
- removed copper zone on B.Cu, net GND2
- removed copper zone on F.Cu, net GND2
- removed copper zone on B.Cu, net GND3
- removed copper zone on F.Cu, net GND3
Other:
- board size 100 x 100 mm -> 100 x 32.7 mm
- board text removed: "Solid pad"
- board text removed: "Thermal reliefs"

Commit message: update
Parts:
- added BZ1: Buzzer, Footprint:LD-BZEN-1205, F.Cu at (150.5, 65.0)
- added R1: 6k2, Resistor_THT:R_Axial_DIN0207_L6.3mm_D2.5mm_P7.62mm_Horizontal, F.Cu at (138.9, 71.1)
- added R2: 390, Resistor_THT:R_Axial_DIN0207_L6.3mm_D2.5mm_P7.62mm_Horizontal, F.Cu at (138.9, 75.2)
- added R3: 910, Resistor_THT:R_Axial_DIN0207_L6.3mm_D2.5mm_P7.62mm_Horizontal, F.Cu at (138.9, 79.2)
- added R4: 1k, Resistor_THT:R_Axial_DIN0207_L6.3mm_D2.5mm_P7.62mm_Horizontal, F.Cu at (138.9, 83.2)
- added R5: 1k1, Resistor_THT:R_Axial_DIN0207_L6.3mm_D2.5mm_P7.62mm_Horizontal, F.Cu at (138.9, 87.3)
- added R6: 620, Resistor_THT:R_Axial_DIN0207_L6.3mm_D2.5mm_P7.62mm_Horizontal, F.Cu at (138.9, 91.3)
- added R7: 1k3, Resistor_THT:R_Axial_DIN0207_L6.3mm_D2.5mm_P7.62mm_Horizontal, F.Cu at (138.9, 95.4)
- added R8: 1k5, Resistor_THT:R_Axial_DIN0207_L6.3mm_D2.5mm_P7.62mm_Horizontal, F.Cu at (138.9, 99.5)
- added R9: 1k, Resistor_THT:R_Axial_DIN0207_L6.3mm_D2.5mm_P7.62mm_Horizontal, F.Cu at (138.9, 103.5)
- added SW10: SW_SPDT, Footprint:OS102011MS2QN1, F.Cu at (155.9, 79.5)
Other:
- board outline removed

Commit message: update
Parts:
- R1, R2, R3, R4, R5, R6, R7, R8, R9: footprint Resistor_THT:R_Axial_DIN0207_L6.3mm_D2.5mm_P7.62mm_Horizontal -> Resistor_THT:R_Axial_DIN0207_L6.3mm_D2.5mm_P10.16mm_Horizontal

Commit message: update
Parts:
- added C1: 100n, Capacitor_THT:C_Disc_D3.0mm_W1.6mm_P2.50mm, F.Cu at (137.9, 59.0)
- added D1: D_Schottky, Diode_THT:D_DO-41_SOD81_P10.16mm_Horizontal, F.Cu at (146.8, 52.2)
- added J1: Barrel Jack, Footprint:DCJ250-10-A-K1-K, F.Cu at (128.4, 51.8)
- added SW1: SW_Push, Button_Switch_THT:SW_PUSH_6mm_H4.3mm, F.Cu at (116.0, 71.8)
- added SW2: SW_Push, Button_Switch_THT:SW_PUSH_6mm_H4.3mm, F.Cu at (116.0, 80.3)
- added SW3: SW_Push, Button_Switch_THT:SW_PUSH_6mm_H4.3mm, F.Cu at (116.0, 88.9)
- added SW4: SW_Push, Button_Switch_THT:SW_PUSH_6mm_H4.3mm, F.Cu at (116.0, 97.5)
- added SW5: SW_Push, Button_Switch_THT:SW_PUSH_6mm_H4.3mm, F.Cu at (116.0, 106.0)
- added SW6: SW_Push, Button_Switch_THT:SW_PUSH_6mm_H4.3mm, F.Cu at (126.5, 71.8)
- added SW7: SW_Push, Button_Switch_THT:SW_PUSH_6mm_H4.3mm, F.Cu at (126.5, 80.3)
- added SW8: SW_Push, Button_Switch_THT:SW_PUSH_6mm_H4.3mm, F.Cu at (126.5, 88.9)
- U1: footprint Package_DIP:DIP-8_W7.62mm -> Footprint:DIP-8_W7.62mm-socket
Connections:
- R9 pad 2: Net-(SW10-A) -> Net-(D1-K)
- SW10 pad 1: Net-(SW10-A) -> Net-(D1-A)
- U1 pad 4: Net-(SW10-A) -> Net-(D1-K)
- U1 pad 8: Net-(SW10-A) -> Net-(D1-K)

Commit message: update
Parts:
- added G***: LOGO, Footprint:piano-silk, F.Cu at (56.0, 168.5)
- added H1: MountingHole_Pad, MountingHole:MountingHole_3.2mm_M3_Pad_Via, F.Cu at (50.0, 80.5)
- added H2: MountingHole_Pad, MountingHole:MountingHole_3.2mm_M3_Pad_Via, F.Cu at (150.0, 80.5)
- added H3: MountingHole_Pad, MountingHole:MountingHole_3.2mm_M3_Pad_Via, F.Cu at (150.0, 180.5)
- added H4: MountingHole_Pad, MountingHole:MountingHole_3.2mm_M3_Pad_Via, F.Cu at (50.0, 180.5)
- BZ1: value Buzzer -> LD-BZEN-1205
- D1: value D_Schottky -> SR150-DC
- moved SW1 107.2 mm to (67.2, 167.2)
- moved SW6 95.7 mm to (120.1, 167.2)
- moved SW2 94.9 mm to (77.8, 167.2)
- moved SW7 87.0 mm to (130.7, 167.2)
- moved SW3 83.1 mm to (88.4, 167.2)
- moved SW8 79.7 mm to (141.2, 167.2)
- moved SW4 71.8 mm to (99.0, 167.2)
- moved SW5 61.6 mm to (109.5, 167.2)
- moved R5 55.7 mm to (121.9, 140.3)
- moved BZ1 55.7 mm to (133.5, 118.0)
- moved C1 55.7 mm to (120.9, 112.0)
- moved D1 55.7 mm to (129.8, 105.2)
- moved J1 55.7 mm to (111.4, 104.8)
- moved R1 55.7 mm to (121.9, 124.1)
- moved R2 55.7 mm to (121.9, 128.2)
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Other:
- board outline added: 108 x 108 mm

Commit message: update
Parts:
- added C2: 470u / 50V, Capacitor_THT:CP_Radial_D10.0mm_P5.00mm, F.Cu at (117.8, 135.6)
- added D2: RED, LED_THT:LED_D5.0mm, F.Cu at (114.2, 83.8)
- added D3: YELLOW, LED_THT:LED_D5.0mm, F.Cu at (131.8, 130.5)
- added D4: GREEN, LED_THT:LED_D5.0mm, F.Cu at (131.8, 137.3)
- added G***: LOGO, Footprint:9V, F.Cu at (64.6, 85.8)
- added G***: LOGO, Footprint:soldering, F.Cu at (136.6, 85.8)
- added G***: LOGO, Footprint:TVZ, F.Cu at (99.4, 111.0)
- added J2: Conn_01x05_Pin, Connector_PinHeader_2.54mm:PinHeader_1x05_P2.54mm_Horizontal, F.Cu at (58.8, 120.2)
- added J3: Conn_01x05_Socket, Connector_PinSocket_2.54mm:PinSocket_1x05_P2.54mm_Vertical, F.Cu at (64.5, 110.0)
- added J4: Conn_01x03_Pin, Connector_PinHeader_2.54mm:PinHeader_1x03_P2.54mm_Vertical, F.Cu at (67.0, 120.2)
- added J5: Conn_01x03_Pin, Connector_PinHeader_2.54mm:PinHeader_1x03_P2.54mm_Vertical, F.Cu at (67.0, 115.1)
- added R10: 4k7, Resistor_THT:R_Axial_DIN0207_L6.3mm_D2.5mm_P10.16mm_Horizontal, F.Cu at (124.2, 80.3)
- added R11: 2k2, Resistor_THT:R_Axial_DIN0207_L6.3mm_D2.5mm_P10.16mm_Horizontal, F.Cu at (112.7, 143.8)
- added R12: 2k2, Resistor_THT:R_Axial_DIN0207_L6.3mm_D2.5mm_P2.54mm_Vertical, F.Cu at (81.9, 110.0)
- added R13: 2k2, Resistor_THT:R_Axial_DIN0207_L6.3mm_D2.5mm_P2.54mm_Vertical, F.Cu at (81.9, 115.1)
- added R14: 2k2, Resistor_THT:R_Axial_DIN0207_L6.3mm_D2.5mm_P2.54mm_Vertical, F.Cu at (81.9, 120.2)
- added SW11: C/D, Footprint:OS102011MS2QN1, F.Cu at (143.8, 135.3)
- added TP1: TestPoint, Footprint:Wire, F.Cu at (130.8, 99.0)
- added TP2: TestPoint, Footprint:Wire, F.Cu at (130.8, 117.2)
- SW10: value SW_SPDT -> POWER
- moved R1 65.9 mm to (56.0, 152.9), turned to -90 degrees
- moved SW10 65.3 mm to (94.2, 85.0), turned to 90 degrees
- moved BZ1 63.5 mm to (75.2, 143.2), turned to 90 degrees
- moved R2 53.5 mm to (68.6, 152.9), turned to -90 degrees
- moved U1 47.2 mm to (88.0, 136.2)
- moved C1 45.5 mm to (93.2, 148.2), turned to 180 degrees
- moved R3 41.6 mm to (81.1, 152.9), turned to -90 degrees
- moved R8 36.3 mm to (144.0, 152.9), turned to -90 degrees
- moved J1 35.2 mm to (79.2, 90.5), turned to 180 degrees
- moved R4 30.9 mm to (93.7, 152.9), turned to -90 degrees
- moved D1 29.6 mm to (104.2, 90.4), turned to 90 degrees
- moved G*** 27.7 mm to (56.6, 140.8)
- moved R7 26.5 mm to (131.4, 152.9), turned to -90 degrees
- moved R5 22.8 mm to (106.3, 152.9), turned to -90 degrees
- moved R9 21.4 mm to (103.8, 145.1), turned to 90 degrees
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- renumbered R8 to R1, R7 to R2, R6 to R3, R5 to R4, R4 to R5, R3 to R6, R2 to R7, R1 to R8
Connections:
- net Net-(D1-K) renamed VDD
Routing:
- net (no net): track 0.00 -> 34.6 mm
Other:
- outline, holes or cut-outs redrawn
- board text added: "CAPACITOR CHARGE/DISCHARGE"
- board text added: "CHARGE"
- board text added: "DISCHARGE"
- board text added: "DUMMY COMPONENTS"
- board text added: "JUMPER WIRE"
- board text added: "OFF"
- board text added: "ON"
- board text added: "PIANO"
- board text added: "POWER"
- board text added: "TVZ THD SolderingPracticeKit V1rev1"

Commit message: update
Parts:
- moved TP2 15.1 mm to (125.4, 103.1), turned to -90 degrees
- moved TP1 13.4 mm to (143.6, 103.1), turned to -90 degrees
Other:
- board text added: "HIGH CURRENT TRACES"
Changed lines of the file:
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@@
 	(footprint "Footprint:Wire"
 		(layer "F.Cu")
-		(at 130.8 117.2)
+		(at 125.4 103.1 -90)
 		(property "Reference" "TP2"
-			(at 0 -2 0)
+			(at 0 -2 270)
 			(unlocked yes)
 			(layer "F.SilkS")
@@
 		)
 		(property "Value" "TestPoint"
-			(at 0 2.5 0)
+			(at 0 2.5 270)
 			(unlocked yes)
 			(layer "F.Fab")
@@
 		)
 		(property "Datasheet" ""
-			(at 0 0 0)
+			(at 0 0 270)
 			(unlocked yes)
 			(layer "F.Fab")
@@
 		)
 		(property "Description" "test point"
-			(at 0 0 0)
+			(at 0 0 270)
 			(unlocked yes)
 			(layer "F.Fab")
@@
 		(attr board_only exclude_from_pos_files)
 		(fp_text user "${REFERENCE}"
-			(at 0 4 0)
+			(at 0 4 270)
 			(unlocked yes)
 			(layer "F.Fab")
@@
 		)
 		(pad "1" thru_hole circle
-			(at 0 0)
+			(at 0 0 270)
 			(size 2.5 2.5)
 			(drill 1.5)
@@
 	(footprint "Footprint:Wire"
 		(layer "F.Cu")
-		(at 130.8 99)
+		(at 143.6 103.1 -90)
 		(property "Reference" "TP1"
-			(at 0 -2 0)
+			(at 0 -2 270)
 			(unlocked yes)
 			(layer "F.SilkS")
@@
 		)
 		(property "Value" "TestPoint"
-			(at 0 2.5 0)
+			(at 0 2.5 270)
 			(unlocked yes)
 			(layer "F.Fab")
@@
 		)
 		(property "Datasheet" ""
-			(at 0 0 0)
+			(at 0 0 270)
 			(unlocked yes)
 			(layer "F.Fab")
@@
 		)
 		(property "Description" "test point"
-			(at 0 0 0)
+			(at 0 0 270)
 			(unlocked yes)
 			(layer "F.Fab")
@@
 		(attr board_only exclude_from_pos_files)
 		(fp_text user "${REFERENCE}"
-			(at 0 4 0)
+			(at 0 4 270)
 			(unlocked yes)
 			(layer "F.Fab")
@@
 		)
 		(pad "1" thru_hole circle
-			(at 0 0)
+			(at 0 0 270)
 			(size 2.5 2.5)
 			(drill 1.5)
@@
 	)
 	(gr_line
-		(start 142.2 100.3)
-		(end 142.2 116.1)
+		(start 142.3 114.5)
+		(end 126.5 114.5)
 		(stroke
 			(width 5)
@@
 	)
 	(gr_line
-		(start 136 98.8)
-		(end 136 117.6)
+		(start 143.8 108.3)
+		(end 125 108.3)
 		(stroke
 			(width 2)
@@
 	)
 	(gr_line
-		(start 130.8 115.4)
-		(end 130.8 113.8)
+		(start 127.2 103.1)
+		(end 128.8 103.1)
 		(stroke
 			(width 0.4)
@@
 	)
 	(gr_line
-		(start 130.8 100.8)
-		(end 130.8 102.6)
+		(start 141.8 103.1)
+		(end 140 103.1)
 		(stroke
 			(width 0.4)
@@
 	)
 	(gr_text "DUMMY COMPONENTS"
-		(at 49.6 102.2 0)
+		(at 49.6 100.528 0)
 		(layer "F.SilkS")
 		(effects
@@
 	)
 	(gr_text "JUMPER WIRE"
-		(at 131.52625 113.546429 90)
+		(at 129.053571 103.82625 0)
 		(layer "F.SilkS")
 		(effects
@@
 		)
 	)
+	(gr_text "HIGH CURRENT TRACES"
+		(at 115 100.528 0)
+		(layer "F.SilkS")
+		(effects
+			(font
+				(size 2 2)
+				(thickness 0.4)
+				(bold yes)
+			)
+			(justify left bottom)
+		)
+	)
 	(gr_text "OFF"
 		(at 84.933333 80.15 0)
@@
 	)
 	(segment
-		(start 136 98.8)
-		(end 136 117.6)
+		(start 143.8 108.3)
+		(end 125 108.3)
 		(width 2)
 		(layer "F.Cu")
@@
 	)
 	(segment
-		(start 142.2 100.3)
-		(end 142.2 116.1)
+		(start 142.3 114.5)
+		(end 126.5 114.5)
 		(width 5)
 		(layer "F.Cu")
