File: KiCAD Files/TVZSolderingPracticeKit.kicad_pcb (KiCad board)
At the start: 2 copper layers, 108 x 108 mm, 47 parts, among them J1 Barrel Jack, J2 Conn_01x05_Pin, J3 Conn_01x05_Socket, J4 Conn_01x03_Pin, J5 Conn_01x03_Pin, SW1 SW_Push, SW10 POWER, SW11 C/D, SW2 SW_Push, SW3 SW_Push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

Commit message: update
Parts:
- moved H1 4.00 mm to (54.0, 80.5)
- moved H2 4.00 mm to (146.0, 80.5)
- moved H3 4.00 mm to (146.0, 180.5)
- moved H4 4.00 mm to (54.0, 180.5)
- moved G*** 3.10 mm to (133.5, 85.8)
- moved J3 2.10 mm to (66.6, 109.9)
- moved J2 2.10 mm to (60.9, 120.1)
- moved J4 2.10 mm to (69.1, 120.1)
- moved J5 2.10 mm to (69.1, 115.0)
- moved R12 2.10 mm to (84.0, 109.9)
- moved R13 2.10 mm to (84.0, 115.0)
- moved R14 2.10 mm to (84.0, 120.1)
Other:
- board size 108 x 108 mm -> 100 x 108 mm
Changed lines of the file:
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@@
 	(footprint "Resistor_THT:R_Axial_DIN0207_L6.3mm_D2.5mm_P2.54mm_Vertical"
 		(layer "F.Cu")
-		(at 81.86 120.17)
+		(at 83.96 120.08)
 		(descr "Resistor, Axial_DIN0207 series, Axial, Vertical, pin pitch=2.54mm, 0.25W = 1/4W, length*diameter=6.3*2.5mm^2, http://cdn-reichelt.de/documents/datenblatt/B400/1_4W%23YAG.pdf")
 		(tags "Resistor Axial_DIN0207 series Axial Vertical pin pitch 2.54mm 0.25W = 1/4W length 6.3mm diameter 2.5mm")
@@
 	(footprint "Resistor_THT:R_Axial_DIN0207_L6.3mm_D2.5mm_P2.54mm_Vertical"
 		(layer "F.Cu")
-		(at 81.86 109.985)
+		(at 83.96 109.895)
 		(descr "Resistor, Axial_DIN0207 series, Axial, Vertical, pin pitch=2.54mm, 0.25W = 1/4W, length*diameter=6.3*2.5mm^2, http://cdn-reichelt.de/documents/datenblatt/B400/1_4W%23YAG.pdf")
 		(tags "Resistor Axial_DIN0207 series Axial Vertical pin pitch 2.54mm 0.25W = 1/4W length 6.3mm diameter 2.5mm")
@@
 	(footprint "Connector_PinHeader_2.54mm:PinHeader_1x03_P2.54mm_Vertical"
 		(layer "F.Cu")
-		(at 67 115.09 90)
+		(at 69.1 115 90)
 		(descr "Through hole straight pin header, 1x03, 2.54mm pitch, single row")
 		(tags "Through hole pin header THT 1x03 2.54mm single row")
@@
 	(footprint "MountingHole:MountingHole_3.2mm_M3_Pad_Via"
 		(layer "F.Cu")
-		(at 150 180.5)
+		(at 146 180.5)
 		(descr "Mounting Hole 3.2mm, M3, generated by kicad-footprint-generator mountinghole.py")
 		(tags "mountinghole M3")
@@
 	(footprint "Resistor_THT:R_Axial_DIN0207_L6.3mm_D2.5mm_P2.54mm_Vertical"
 		(layer "F.Cu")
-		(at 81.86 115.09)
+		(at 83.96 115)
 		(descr "Resistor, Axial_DIN0207 series, Axial, Vertical, pin pitch=2.54mm, 0.25W = 1/4W, length*diameter=6.3*2.5mm^2, http://cdn-reichelt.de/documents/datenblatt/B400/1_4W%23YAG.pdf")
 		(tags "Resistor Axial_DIN0207 series Axial Vertical pin pitch 2.54mm 0.25W = 1/4W length 6.3mm diameter 2.5mm")
@@
 	(footprint "Footprint:soldering"
 		(layer "F.Cu")
-		(at 136.6 85.806371)
+		(at 133.5 85.806371)
 		(property "Reference" "G***"
 			(at 0 0 0)
@@
 	(footprint "Connector_PinHeader_2.54mm:PinHeader_1x03_P2.54mm_Vertical"
 		(layer "F.Cu")
-		(at 67 120.17 90)
+		(at 69.1 120.08 90)
 		(descr "Through hole straight pin header, 1x03, 2.54mm pitch, single row")
 		(tags "Through hole pin header THT 1x03 2.54mm single row")
@@
 	(footprint "Connector_PinHeader_2.54mm:PinHeader_1x05_P2.54mm_Horizontal"
 		(layer "F.Cu")
-		(at 58.785 120.17 180)
+		(at 60.885 120.08 180)
 		(descr "Through hole angled pin header, 1x05, 2.54mm pitch, 6mm pin length, single row")
 		(tags "Through hole angled pin header THT 1x05 2.54mm single row")
@@
 	(footprint "MountingHole:MountingHole_3.2mm_M3_Pad_Via"
 		(layer "F.Cu")
-		(at 50 80.5)
+		(at 54 80.5)
 		(descr "Mounting Hole 3.2mm, M3, generated by kicad-footprint-generator mountinghole.py")
 		(tags "mountinghole M3")
@@
 	(footprint "Connector_PinSocket_2.54mm:PinSocket_1x05_P2.54mm_Vertical"
 		(layer "F.Cu")
-		(at 64.46 109.985 90)
+		(at 66.56 109.895 90)
 		(descr "Through hole straight socket strip, 1x05, 2.54mm pitch, single row (from Kicad 4.0.7), script generated")
 		(tags "Through hole socket strip THT 1x05 2.54mm single row")
@@
 	(footprint "MountingHole:MountingHole_3.2mm_M3_Pad_Via"
 		(layer "F.Cu")
-		(at 50 180.5)
+		(at 54 180.5)
 		(descr "Mounting Hole 3.2mm, M3, generated by kicad-footprint-generator mountinghole.py")
 		(tags "mountinghole M3")
@@
 	(footprint "MountingHole:MountingHole_3.2mm_M3_Pad_Via"
 		(layer "F.Cu")
-		(at 150 80.5)
+		(at 146 80.5)
 		(descr "Mounting Hole 3.2mm, M3, generated by kicad-footprint-generator mountinghole.py")
 		(tags "mountinghole M3")
@@
 	(gr_line
 		(start 110.2 120)
-		(end 149.6 120)
+		(end 148 120)
 		(stroke
 			(width 0.3)
@@
 	)
 	(gr_line
-		(start 50.2 128.6)
+		(start 52 128.6)
 		(end 101.6 128.6)
 		(stroke
@@
 	)
 	(gr_line
-		(start 50.2 96.4)
-		(end 149.6 96.4)
+		(start 52 96.4)
+		(end 148 96.4)
 		(stroke
 			(width 0.3)
@@
 	)
 	(gr_line
-		(start 149.6 148.2)
+		(start 148 148.2)
 		(end 110.2 148.2)
 		(stroke
@@
 	)
 	(gr_arc
-		(start 154 180.5)
-		(mid 152.828427 183.328427)
-		(end 150 184.5)
+		(start 150 180.5)
+		(mid 148.828427 183.328427)
+		(end 146 184.5)
 		(stroke
 			(width 0.05)
@@
 	)
 	(gr_line
-		(start 46 86)
-		(end 46 80.5)
+		(start 146 184.5)
+		(end 54 184.5)
 		(stroke
 			(width 0.05)
@@
 	)
 	(gr_line
-		(start 154 175)
-		(end 154 180.5)
+		(start 50 80.5)
+		(end 50 180.5)
 		(stroke
 			(width 0.05)
@@
 	)
 	(gr_line
-		(start 150 184.5)
-		(end 50 184.5)
-		(stroke
-			(width 0.05)
-			(type default)
-		)
-		(layer "Edge.Cuts")
-	)
-	(gr_line
-		(start 48 88)
-		(end 48 173)
-		(stroke
-			(width 0.05)
-			(type default)
-		)
-		(layer "Edge.Cuts")
-	)
-	(gr_line
-		(start 48 88)
-		(end 46 86)
-		(stroke
-			(width 0.05)
-			(type default)
-		)
-		(layer "Edge.Cuts")
-	)
-	(gr_line
-		(start 150 76.5)
-		(end 50 76.5)
-		(stroke
-			(width 0.05)
-			(type default)
-		)
-		(layer "Edge.Cuts")
-	)
-	(gr_line
-		(start 46 175)
-		(end 46 180.5)
-		(stroke
-			(width 0.05)
-			(type default)
-		)
-		(layer "Edge.Cuts")
-	)
-	(gr_line
-		(start 46 175)
-		(end 48 173)
-		(stroke
-			(width 0.05)
-			(type default)
-		)
-		(layer "Edge.Cuts")
-	)
-	(gr_line
-		(start 152 173)
-		(end 154 175)
+		(start 146 76.5)
+		(end 54 76.5)
 		(stroke
 			(width 0.05)
@@
 	)
 	(gr_arc
-		(start 50 184.5)
-		(mid 47.171573 183.328427)
-		(end 46 180.5)
+		(start 54 184.5)
+		(mid 51.171573 183.328427)
+		(end 50 180.5)
 		(stroke
 			(width 0.05)
@@
 	)
 	(gr_arc
-		(start 46 80.5)
-		(mid 47.171573 77.671573)
-		(end 50 76.5)
-		(stroke
-			(width 0.05)
-			(type default)
-		)
-		(layer "Edge.Cuts")
-	)
-	(gr_line
-		(start 154 86)
-		(end 154 80.5)
+		(start 50 80.5)
+		(mid 51.171573 77.671573)
+		(end 54 76.5)
 		(stroke
 			(width 0.05)
@@
 	)
 	(gr_line
-		(start 154 86)
-		(end 152 88)
+		(start 150 86)
+		(end 150 80.5)
 		(stroke
 			(width 0.05)
@@
 	)
 	(gr_line
-		(start 152 173)
-		(end 152 88)
+		(start 150 180.5)
+		(end 150 86)
 		(stroke
 			(width 0.05)
@@
 	)
 	(gr_arc
-		(start 150 76.5)
-		(mid 152.828427 77.671573)
-		(end 154 80.5)
+		(start 146 76.5)
+		(mid 148.828427 77.671573)
+		(end 150 80.5)
 		(stroke
 			(width 0.05)
@@
 	)
 	(gr_text "DUMMY COMPONENTS"
-		(at 49.6 100.528 0)
+		(at 51.5 100.5 0)
 		(layer "F.SilkS")
 		(effects
@@
 	)
 	(gr_text "HIGH CURRENT TRACES"
-		(at 115 100.528 0)
+		(at 113.5 100.5 0)
 		(layer "F.SilkS")
 		(effects

Commit message: update
Parts:
- moved C1 17.2 mm to (93.2, 131.0)
- moved D1 4.00 mm to (104.2, 94.4)
- moved D2 4.00 mm to (114.2, 87.8)
- moved G*** 4.00 mm to (64.6, 89.8)
- moved G*** 4.00 mm to (133.5, 89.8)
- moved H1 4.00 mm to (54.0, 84.5)
- moved H2 4.00 mm to (146.0, 84.5)
- moved H3 4.00 mm to (146.0, 176.5)
- moved H4 4.00 mm to (54.0, 176.5)
- moved J1 4.00 mm to (79.2, 94.5)
- moved R10 4.00 mm to (124.2, 84.3)
- moved SW10 4.00 mm to (94.2, 89.0)
- moved SW1 3.87 mm to (52.8, 163.4)
- moved SW2 3.87 mm to (65.3, 163.4)
- moved SW3 3.87 mm to (77.9, 163.4)
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Other:
- board size 100 x 108 mm -> 100 x 100 mm

Commit message: update
Parts:
- removed the G*** at (133.5, 89.8)
- removed the G*** at (99.4, 111.0)
- added G***: LOGO, Footprint:TVZ-15mm, F.Cu at (136.0, 91.5)
- moved J2 79.3 mm to (139.1, 106.9), turned to 0 degrees
- moved TP2 70.5 mm to (55.3, 110.3)
- moved TP1 69.0 mm to (75.0, 110.3)
- moved J3 67.3 mm to (133.4, 117.1), turned to -90 degrees
- moved J4 63.2 mm to (130.9, 106.9), turned to -90 degrees
- moved J5 61.9 mm to (130.9, 112.0), turned to -90 degrees
- moved R14 35.6 mm to (117.0, 106.9), turned to 180 degrees
- moved R12 33.9 mm to (117.0, 117.1), turned to 180 degrees
- moved R13 33.2 mm to (117.0, 112.0), turned to 180 degrees
- moved G*** 2.89 mm to (56.6, 137.9)
- moved D2 2.23 mm to (114.2, 90.0)
- moved R10 2.23 mm to (124.2, 86.5)
- moved SW10 2.23 mm to (94.2, 91.2)
- moved D1 2.23 mm to (104.2, 96.7)
- moved R11 2.10 mm to (112.7, 141.7)
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Routing:
- net VDD: track 0.00 -> 180.1 mm
- net Net-(U1-THR): track 0.00 -> 110.1 mm
- net Net-(U1-DIS): track 0.00 -> 53.3 mm
- net unconnected-(H1-Pad1): track 0.00 -> 38.0 mm
- net (no net): track 34.6 -> 0.00 mm
- net Net-(R3-Pad1): track 0.00 -> 30.0 mm
- net Net-(R4-Pad1): track 0.00 -> 29.9 mm
- net Net-(R5-Pad1): track 0.00 -> 29.9 mm
- net Net-(R2-Pad1): track 0.00 -> 29.9 mm
- net Net-(R6-Pad1): track 0.00 -> 29.8 mm
- net Net-(R7-Pad1): track 0.00 -> 29.8 mm
- net Net-(R1-Pad1): track 0.00 -> 29.8 mm
- net Net-(SW11-B): track 0.00 -> 24.4 mm
- net Net-(D3-A): track 0.00 -> 19.3 mm
- net Net-(SW10-B): track 0.00 -> 17.1 mm
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- added copper zone on B.Cu, net GND1
- added copper zone on F.Cu, net GND1
Other:
- outline, holes or cut-outs redrawn
- board text added: "THD Interactive Soldering Practice Kit V1rev1"
- board text removed: "TVZ THD SolderingPracticeKit V1rev1"

Commit message: update
Parts:
- added D5: WHITE, LED_THT:LED_D5.0mm, F.Cu at (94.2, 121.3)
- added G***: LOGO, Footprint:logo, B.Cu at (64.8, 173.6)
- added R15: 2k2, Resistor_THT:R_Axial_DIN0207_L6.3mm_D2.5mm_P10.16mm_Horizontal, F.Cu at (104.2, 117.1)
- added RV1: 10k, Footprint:RK09K1130AH1, F.Cu at (91.7, 118.0)
- moved TP2 1.65 mm to (56.9, 109.9)
- moved TP1 1.65 mm to (76.6, 109.9)
Routing:
- net Net-(R15-Pad2): track 0.00 -> 19.7 mm
- net VDD: track 180.1 -> 199.0 mm
- net Net-(D5-A): track 0.00 -> 12.8 mm
Other:
- board text added: "JLCJLCJLCJLC"

Commit message: update
Parts:
- moved G*** 69.8 mm to (134.6, 172.6)
Other:
- board text added: "github.com/jkordek1/TVZSolderingPracticeKit"
Changed lines of the file:
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@@
 	(footprint "Footprint:logo"
 		(layer "B.Cu")
-		(at 64.8 173.6 180)
+		(at 134.6 172.6 180)
 		(property "Reference" "G***"
 			(at 0 0 0)
@@
 	)
 	(gr_text "JLCJLCJLCJLC"
-		(at 137.6 177.6 0)
+		(at 74.4 176.93775 0)
 		(layer "B.SilkS")
 		(effects
@@
 			)
 			(justify left bottom mirror)
+		)
+	)
+	(gr_text "github.com/jkordek1/TVZSolderingPracticeKit"
+		(at 137.8 177 0)
+		(layer "B.SilkS")
+		(effects
+			(font
+				(size 1.2 1.2)
+				(thickness 0.2)
+				(bold yes)
+			)
+			(justify left bottom mirror)

Commit message: update
Connections:
- RV1 pad 1: unconnected-(RV1-Pad1) -> Net-(R15-Pad2)
Routing:
- net Net-(R15-Pad2): track 19.7 -> 22.2 mm
Changed lines of the file:
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@@
 	(net 67 "unconnected-(TP1-Pad1)")
 	(net 68 "unconnected-(TP2-Pad1)")
-	(net 69 "unconnected-(RV1-Pad1)")
-	(net 70 "Net-(D5-A)")
-	(net 71 "Net-(R15-Pad2)")
+	(net 69 "Net-(D5-A)")
+	(net 70 "Net-(R15-Pad2)")
 	(footprint "Resistor_THT:R_Axial_DIN0207_L6.3mm_D2.5mm_P2.54mm_Vertical"
 		(layer "F.Cu")
@@
 		(tags "Through hole pin header THT 1x03 2.54mm single row")
 		(property "Reference" "J5"
-			(at 0 -2.38 180)
+			(at 0 -2.38 0)
 			(layer "F.SilkS")
 			(effects
@@
 			)
 		)
+		(property "TME Part Number" "ZL201-03G"
+			(at 0 0 270)
+			(unlocked yes)
+			(layer "F.Fab")
+			(hide yes)
+			(effects
+				(font
+					(size 1 1)
+					(thickness 0.15)
+				)
+			)
+		)
 		(property ki_fp_filters "Connector*:*_1x??_*")
 		(sheetname "/")
@@
 		)
 		(embedded_fonts no)
-		(model "${KICAD9_3DMODEL_DIR}/Connector_PinHeader_2.54mm.3dshapes/PinHeader_1x03_P2.54mm_Vertical.wrl"
+		(model "${KIPRJMOD}/Component3DModels/pinheader 1x3 and 1 jumper pullback black.step"
 			(offset
-				(xyz 0 0 0)
+				(xyz -11 17.5 0)
 			)
 			(scale
@@
 			)
 			(rotate
-				(xyz 0 0 0)
+				(xyz -0 -0 90)
 			)
 		)
@@
 			(layers "*.Cu" "*.Mask")
 			(remove_unused_layers no)
-			(net 69 "unconnected-(RV1-Pad1)")
+			(net 70 "Net-(R15-Pad2)")
 			(pinfunction "1")
-			(pintype "passive+no_connect")
+			(pintype "passive")
 		)
 		(pad "2" thru_hole circle
@@
 			(layers "*.Cu" "*.Mask")
 			(remove_unused_layers no)
-			(net 71 "Net-(R15-Pad2)")
+			(net 70 "Net-(R15-Pad2)")
 			(pinfunction "2")
 			(pintype "passive")
@@
 		(tags "Through hole pin header THT 1x03 2.54mm single row")
 		(property "Reference" "J4"
-			(at 0 -2.38 180)
+			(at 0 -2.38 0)
 			(layer "F.SilkS")
 			(effects
@@
 			)
 		)
+		(property "TME Part Number" "ZL201-03G"
+			(at 0 0 270)
+			(unlocked yes)
+			(layer "F.Fab")
+			(hide yes)
+			(effects
+				(font
+					(size 1 1)
+					(thickness 0.15)
+				)
+			)
+		)
 		(property ki_fp_filters "Connector*:*_1x??_*")
 		(sheetname "/")
@@
 		)
 		(embedded_fonts no)
-		(model "${KICAD9_3DMODEL_DIR}/Connector_PinHeader_2.54mm.3dshapes/PinHeader_1x03_P2.54mm_Vertical.wrl"
+		(model "${KIPRJMOD}/Component3DModels/pinheader 1x3 and 1 jumper pullback.stp"
 			(offset
-				(xyz 0 0 0)
+				(xyz -11 17.5 0)
 			)
 			(scale
@@
 			)
 			(rotate
-				(xyz 0 0 0)
+				(xyz -0 -0 90)
 			)
 		)
@@
 		(tags "LED")
 		(property "Reference" "D3"
-			(at 1.27 4.3 180)
+			(at 1.27 4.3 0)
 			(layer "F.SilkS")
 			(effects
@@
 		)
 		(embedded_fonts no)
-		(model "${KICAD9_3DMODEL_DIR}/LED_THT.3dshapes/LED_D5.0mm.wrl"
+		(model "${KIPRJMOD}/Component3DModels/LED_Round_Yellow_D5.0mm.step"
 			(offset
 				(xyz 0 0 0)
@@
 			(layers "*.Cu" "*.Mask")
 			(remove_unused_layers no)
-			(net 70 "Net-(D5-A)")
+			(net 69 "Net-(D5-A)")
 			(pinfunction "A")
 			(pintype "passive")
 		)
 		(embedded_fonts no)
-		(model "${KICAD9_3DMODEL_DIR}/LED_THT.3dshapes/LED_D5.0mm.wrl"
+		(model "${KIPRJMOD}/Component3DModels/LED_Round_Clear_D5.0mm.step"
 			(offset
 				(xyz 0 0 0)
@@
 			)
 		)
+		(property "TME Part Number" "PH1RB-40-UA"
+			(at 0 0 0)
+			(unlocked yes)
+			(layer "F.Fab")
+			(hide yes)
+			(effects
+				(font
+					(size 1 1)
+					(thickness 0.15)
+				)
+			)
+		)
 		(property ki_fp_filters "Connector*:*_1x??_*")
 		(sheetname "/")
@@
 			(layers "*.Cu" "*.Mask")
 			(remove_unused_layers no)
-			(net 70 "Net-(D5-A)")
+			(net 69 "Net-(D5-A)")
 			(pintype "passive")
 		)
@@
 			(layers "*.Cu" "*.Mask")
 			(remove_unused_layers no)
-			(net 71 "Net-(R15-Pad2)")
+			(net 70 "Net-(R15-Pad2)")
 			(pintype "passive")
 		)
@@
 		(tags "LED")
 		(property "Reference" "D4"
-			(at 1.275 4.3 180)
+			(at 1.275 4.3 0)
 			(layer "F.SilkS")
 			(effects
@@
 		)
 		(embedded_fonts no)
-		(model "${KICAD9_3DMODEL_DIR}/LED_THT.3dshapes/LED_D5.0mm.wrl"
+		(model "${KIPRJMOD}/Component3DModels/LED_Round_Green1_D5.0mm.step"
 			(offset
 				(xyz 0 0 0)
@@
 		(sheetname "/")
 		(sheetfile "TVZSolderingPracticeKit.kicad_sch")
-		(attr board_only exclude_from_pos_files)
+		(attr board_only exclude_from_pos_files exclude_from_bom)
 		(fp_text user "${REFERENCE}"
 			(at 0 4 270)
@@
 			)
 		)
+		(property "TME Part Number" "ZL262-5SG"
+			(at 0 0 270)
+			(unlocked yes)
+			(layer "F.Fab")
+			(hide yes)
+			(effects
+				(font
+					(size 1 1)
+					(thickness 0.15)
+				)
+			)
+		)
 		(property ki_fp_filters "Connector*:*_1x??_*")
 		(sheetname "/")
@@
 		(sheetname "/")
 		(sheetfile "TVZSolderingPracticeKit.kicad_sch")
-		(attr board_only exclude_from_pos_files)
+		(attr board_only exclude_from_pos_files exclude_from_bom)
 		(fp_text user "${REFERENCE}"
 			(at 0 4 270)
@@
 		)
 	)
+	(dimension
+		(type orthogonal)
+		(layer "User.1")
+		(pts
+			(xy 50 84.5) (xy 150 84.5)
+		)
+		(height -8.9)
+		(orientation 0)
+		(format
+			(prefix "")
+			(suffix "")
+			(units 3)
+			(units_format 0)
+			(precision 4)
+			(suppress_zeroes yes)
+		)
+		(style
+			(thickness 0.1)
+			(arrow_length 1.27)
+			(text_position_mode 0)
+			(arrow_direction outward)
+			(extension_height 0.58642)
+			(extension_offset 0.5)
+			(keep_text_aligned yes)
+		)
+		(gr_text "100"
+			(at 100 73.2 0)
+			(layer "User.1")
+			(effects
+				(font
+					(size 2 2)
+					(thickness 0.4)
+					(bold yes)
+				)
+			)
+		)
+	)
+	(dimension
+		(type orthogonal)
+		(layer "User.1")
+		(pts
+			(xy 146 80.5) (xy 146 180.5)
+		)
+		(height 10.4)
+		(orientation 1)
+		(format
+			(prefix "")
+			(suffix "")
+			(units 3)
+			(units_format 0)
+			(precision 4)
+			(suppress_zeroes yes)
+		)
+		(style
+			(thickness 0.1)
+			(arrow_length 1.27)
+			(text_position_mode 0)
+			(arrow_direction outward)
+			(extension_height 0.58642)
+			(extension_offset 0.5)
+			(keep_text_aligned yes)
+		)
+		(gr_text "100"
+			(at 154 130.5 90)
+			(layer "User.1")
+			(effects
+				(font
+					(size 2 2)
+					(thickness 0.4)
+					(bold yes)
+				)
+			)
+		)
+	)
 	(segment
 		(start 147.25 167.88)
@@
 		(width 1)
 		(layer "B.Cu")
-		(net 70)
+		(net 69)
 	)
 	(segment
@@
 		(width 1)
 		(layer "B.Cu")
+		(net 69)
+	)
+	(segment
+		(start 91.7 118.05)
+		(end 94.2 118.05)
+		(width 1)
+		(layer "B.Cu")
 		(net 70)
 	)
@@
 		(width 1)
 		(layer "B.Cu")
-		(net 71)
+		(net 70)
 	)
 	(segment
@@
 		(width 1)
 		(layer "B.Cu")
-		(net 71)
+		(net 70)
 	)
 	(segment
@@
 		(width 1)
 		(layer "B.Cu")
-		(net 71)
+		(net 70)
 	)
 	(zone

Commit message: update
Parts:
- added G***: LOGO, Footprint:soldering-17,5-fab, F.Cu at (47.6, 109.8)
